Commit message: Fix for rotor speed
"time_constant" parameter is not used but "time_constant_up" and "time_constant_down" , time_constant still left not to make problems

File: morus_description/urdf/morus.urdf.xacro (robot description, xacro)
@@ -16,7 +16,13 @@
   <xacro:property name="motor_constant" value="0.000456874" /> <!-- [kg*m/s^2] -->
   <xacro:property name="moment_constant" value="0.01" /> <!-- [m] -->
-  <xacro:property name="time_constant" value="0.125" /> <!-- [s] -->s ti
+  <xacro:property name="time_constant" value="0.125" /> <!-- [s] -->
+  <!-- added time constants for rotos, TODO check -->
+  <!-- change: removed "time_constant" and added "time_constant_down" and "time_constant_up" -->
+  <xacro:property name="time_constant_up"   value="0.25" /> <!-- [s] -->
+  <xacro:property name="time_constant_down" value="0.25" /> <!-- [s] -->
   <xacro:property name="max_rot_velocity" value="838" /> <!-- [rad/s] -->
-  <xacro:property name="rotor_drag_coefficient" value="8.06428e-04" />
+  <!-- Value changed not to have masses getting diverse -->
+  <!-- xacro:property name="rotor_drag_coefficient" value="8.06428e-04" -->
+  <xacro:property name="rotor_drag_coefficient" value="0.0" />
   <xacro:property name="rolling_moment_coefficient" value="0.00001" />
   <xacro:property name="movable_mass_mass" value="1" />
@@ -79,4 +85,6 @@
     radius_rotor="${radius_rotor}"
     time_constant="${time_constant}"
+    time_constant_up="${time_constant_up}"
+    time_constant_down="${time_constant_down}"
     max_rot_velocity="${max_rot_velocity}"
     motor_number="0"
@@ -97,4 +105,6 @@
     radius_rotor="${radius_rotor}"
     time_constant="${time_constant}"
+    time_constant_up="${time_constant_up}"
+    time_constant_down="${time_constant_down}"
     max_rot_velocity="${max_rot_velocity}"
     motor_number="1"
@@ -115,4 +125,6 @@
     radius_rotor="${radius_rotor}"
     time_constant="${time_constant}"
+    time_constant_up="${time_constant_up}"
+    time_constant_down="${time_constant_down}"
     max_rot_velocity="${max_rot_velocity}"
     motor_number="2"
@@ -133,4 +145,6 @@
     radius_rotor="${radius_rotor}"
     time_constant="${time_constant}"
+    time_constant_up="${time_constant_up}"
+    time_constant_down="${time_constant_down}"
     max_rot_velocity="${max_rot_velocity}"
     motor_number="3"

File: morus_description/urdf/multirotor_base.urdf.xacro (robot description, xacro)
@@ -95,6 +95,6 @@
   </xacro:macro>
   <!-- Rotor joint and link -->
-  <xacro:macro name="vertical_rotor"
-    params="robot_namespace suffix direction motor_constant moment_constant parent mass_rotor radius_rotor time_constant max_rot_velocity motor_number rotor_drag_coefficient rolling_moment_coefficient color *origin *inertia">
+   <xacro:macro name="vertical_rotor"
+    params="robot_namespace suffix direction motor_constant moment_constant parent mass_rotor radius_rotor time_constant time_constant_up time_constant_down max_rot_velocity motor_number rotor_drag_coefficient rolling_moment_coefficient color *origin *inertia">
     <joint name="rotor_${motor_number}_joint" type="continuous">
       <xacro:insert_block name="origin" />
@@ -133,4 +133,6 @@
         <turningDirection>${direction}</turningDirection>
         <timeConstant>${time_constant}</timeConstant>
+        <timeConstantUp>${time_constant_up}</timeConstantUp>
+        <timeConstantDown>${time_constant_down}</timeConstantDown>
         <maxRotVelocity>${max_rot_velocity}</maxRotVelocity>
         <motorConstant>${motor_constant}</motorConstant>

Commit message: FIxed offset of moving masses

File: morus_description/urdf/morus.urdf.xacro (robot description, xacro)
@@ -29,5 +29,5 @@
   <xacro:property name="movable_mass_mass" value="1" />
   <xacro:property name="movable_mass_dimension" value="0.08" />
-  <xacro:property name="movable_mass_offset" value="0.025" />
+  <xacro:property name="movable_mass_offset" value="0.05" />
   <xacro:property name="imu_mass" value="0.02"/>
   <xacro:property name="imu_size" value="0.01"/>

Commit message: Functional MPC with moving masses and rotors
All changes to make combined MPC working

File: morus_description/urdf/morus.urdf.xacro (robot description, xacro)
@@ -24,6 +24,6 @@
   <!-- Value changed not to have masses getting diverse -->
   <!-- Enable the drag coefficient -->
-  <!-- xacro:property name="rotor_drag_coefficient" value="8.06428e-04" -->
-  <xacro:property name="rotor_drag_coefficient" value="0.0" />
+  <xacro:property name="rotor_drag_coefficient" value="8.06428e-04" />
+  <!-- xacro:property name="rotor_drag_coefficient" value="0.0" -->
   <xacro:property name="rolling_moment_coefficient" value="0.00001" />
   <xacro:property name="movable_mass_mass" value="1" />
